Commit message: fix robot2

File: xacro/dtw_robot2.xacro (robot description, xacro)
@@ -14,4 +14,9 @@
     </joint>
     <link name="${prefix}_link">
+      <inertial>
+        <origin xyz="0.0 0.0 0.0" rpy="0.0 0.0 0.0"/>
+        <mass value="0.1"/>
+        <inertia ixx="0.0001" ixy="0.0" ixz="0.0" iyy="0.0001" iyz="0.0" izz="0.0001"/>
+      </inertial>
       <visual>
         <geometry>
@@ -20,5 +25,15 @@
         <material name="red"/>
       </visual>
+      <collision>
+        <geometry>
+          <cylinder radius="0.05" length="0.02"/>
+        </geometry>
+      </collision>
     </link>
+    <gazebo reference="${prefix}_link">
+      <material>
+        Gazebo/Red
+      </material>
+    </gazebo>
   </xacro:macro>
   <link name="base_link"/>
@@ -29,4 +44,9 @@
   </joint>
   <link name="body_link">
+    <inertial>
+      <origin xyz="0.0 0.0 0.0" rpy="0.0 0.0 0.0"/>
+      <mass value="1.0"/>
+      <inertia ixx="0.001" ixy="0.0" ixz="0.0" iyy="0.001" iyz="0.0" izz="0.001"/>
+    </inertial>
     <visual>
       <origin xyz="0.0 0.0 0.0" rpy="0.0 0.0 0.0"/>
@@ -36,5 +56,16 @@
       <material name="grey"/>
     </visual>
+    <collision>
+      <origin xyz="0.0 0.0 0.0" rpy="0.0 0.0 0.0"/>
+      <geometry>
+        <box size="0.24 0.178 0.06"/>
+      </geometry>
+    </collision>
   </link>
+  <gazebo reference="body_link">
+    <material>
+      Gazebo/Gray
+    </material>
+  </gazebo>
   <xacro:wheel_macro prefix="left_wheel" parent="base_link" xyz="0 0.1 0.05"/>
   <xacro:wheel_macro prefix="right_wheel" parent="base_link" xyz="0 -0.1 0.05"/>
@@ -52,4 +83,15 @@
       <material name="grey"/>
     </visual>
+    <collision>
+      <origin xyz="0.0 0.0 0.0" rpy="0.0 0.0 0.0"/>
+      <geometry>
+        <sphere radius="0.04"/>
+      </geometry>
+    </collision>
   </link>
+  <gazebo reference="ball_link">
+    <material>
+      Gazebo/Gray
+    </material>
+  </gazebo>
 </robot>
